Commit message: Added PID (steering joint and elevation joint, position joints) for fixing an issue with the gravity. Changed gazebo conditions.

File: hr_recycler_common/hr_recycler_description/urdf/bases/hr_recycler.urdf.xacro (robot description, xacro)
@@ -9,5 +9,6 @@
   <xacro:property name="base_width" value="0.754" />
   <xacro:property name="base_height" value="0.533" />
-  <xacro:property name="base_mass" value="50.0"/>
+  <xacro:property name="base_mass" value="20.0"/>
+  <!--xacro:property name="base_mass" value="50.0"/-->
   <xacro:property name="visual_base_link_z" value="${wheel_radius+base_height/2.0+separation_wheel_box}" />
   <xacro:property name="fork_length" value="1.176" />
@@ -39,5 +40,5 @@
     <inertial>
       <mass value="${base_mass}" />
-      <origin xyz="0 0 0" />
+      <origin xyz="0 0 ${visual_base_link_z}" />
       <box_inertia  m="${base_mass}" x="${base_length}" y="${base_width}" z="${base_height}"/>
     </inertial>

File: hr_recycler_common/hr_recycler_description/urdf/elevator/both_elevator.urdf.xacro (robot description, xacro)
@@ -88,5 +88,5 @@
       <inertial>
         <mass value="${fork_mass}" />
-        <origin xyz="-1 0 0" />
+        <origin xyz="0 0 0" />
         <solid_cuboid_inertia m="${fork_mass}" h="${fork_height}" d="${fork_length}" w="${fork_width}"/>
       </inertial>
@@ -124,5 +124,5 @@
       <inertial>
         <mass value="${fork_mass}" />
-        <origin xyz="-1 0 0" />
+        <origin xyz="0 0 0" />
         <solid_cuboid_inertia m="${fork_mass}" h="${fork_height}" d="${fork_length}" w="${fork_width}"/>
       </inertial>

File: hr_recycler_common/hr_recycler_description/urdf/elevator/elevator.gazebo.xacro (robot description, xacro)
@@ -3,6 +3,6 @@
 	<xacro:macro name="elevator_gazebo" params="prefix">
 		<gazebo reference="${prefix}platform_link">
-			<mu1 value="5.0"/>
-			<mu2 value="0.5"/>
+			<mu1 value="0"/>
+			<mu2 value="0"/>
 			<kp value="10000000.0" />
 			<kd value="1.0" />
@@ -25,27 +25,4 @@
 			<turnGravityOff>false</turnGravityOff-->
 		</gazebo>
-		<gazebo reference="${prefix}_support_wheel_link">
-			<mu1 value="5.0"/>
-			<mu2 value="0.5"/>
-			<kp value="10000000.0" />
-			<kd value="1.0" />
-			<fdir1 value="1 0 0"/>
-			<material>Gazebo/Grey</material>
-			<turnGravityOff>false</turnGravityOff>
-			<kp>500000.0</kp>
-			<kd>10.0</kd>
-			<mu1>0.2</mu1>
-			<mu2>0.2</mu2>
-			<fdir1>1 0 0</fdir1>
-			<!--minDepth>0.001</minDepth-->
-			<!--material>Gazebo/Black</material-->
-			<!--mu1 value="10"/>
-			<mu2 value="5"/>
-			<kp value="500000.0" />
-			<kd value="10.0" />
-			<fdir1 value="1 0 0"/>
-			<material>Gazebo/Yellow</material>
-			<turnGravityOff>false</turnGravityOff-->
-		</gazebo>
 	</xacro:macro>
 </robot>

File: hr_recycler_common/hr_recycler_description/urdf/elevator/elevator.urdf.xacro (robot description, xacro)
@@ -65,4 +65,22 @@
 		</inertial>
 	</link>
+	<gazebo reference="${prefix}_platform_link">
+		<fdir1 value="1 0 0"/>
+		<material>Gazebo/Grey</material>
+		<turnGravityOff>false</turnGravityOff>
+		<kp>500000.0</kp>
+		<kd>100000.0</kd>
+		<mu1>0</mu1>
+		<mu2>0</mu2>
+		<!--minDepth>0.001</minDepth-->
+		<!--material>Gazebo/Black</material-->
+		<!--mu1 value="10"/>
+		<mu2 value="5"/>
+		<kp value="500000.0" />
+		<kd value="10.0" />
+		<fdir1 value="1 0 0"/>
+		<material>Gazebo/Yellow</material>
+		<turnGravityOff>false</turnGravityOff-->
+	</gazebo>
 	<joint name="${prefix}_support_wheel_joint" type="continuous">
 			<origin xyz="${support_wheel_joint_x} ${support_wheel_joint_y} ${support_wheel_joint_z}" rpy="0 0 0"/>
@@ -102,8 +120,22 @@
 	</link>
 	<gazebo reference="${prefix}_support_wheel_link">
-    <mu1>10</mu1>
-    <mu2>10</mu2>
-    <material>Gazebo/Black</material>
-  </gazebo>
+		<fdir1 value="1 0 0"/>
+		<material>Gazebo/Grey</material>
+		<turnGravityOff>false</turnGravityOff>
+		<kp>500000.0</kp>
+		<kd>100000.0</kd>
+		<mu1>0.2</mu1>
+		<mu2>0.2</mu2>
+		<fdir1>1 0 0</fdir1>
+		<!--minDepth>0.001</minDepth-->
+		<!--material>Gazebo/Black</material-->
+		<!--mu1 value="10"/>
+		<mu2 value="5"/>
+		<kp value="500000.0" />
+		<kd value="10.0" />
+		<fdir1 value="1 0 0"/>
+		<material>Gazebo/Yellow</material>
+		<turnGravityOff>false</turnGravityOff-->
+	</gazebo>
 	<!--xacro:elevator_transmission prefix="${prefix}" /-->
 	<!--xacro:elevator_gazebo prefix="${prefix}" /-->

File: hr_recycler_common/hr_recycler_description/urdf/wheels/motor_wheel.urdf.xacro (robot description, xacro)
@@ -7,17 +7,16 @@
   <xacro:property name="wheel_mass" value="5.0" />
   <!-- in kg-->
-  <xacro:property name="steer_joint_damping" value="2000.0" />
-  <xacro:property name="steer_joint_friction" value="1000.0" />
-  <xacro:property name="steer_joint_effort_limit" value="9999.0" />
-  <xacro:property name="steer_joint_velocity_limit" value="200" />
+  <xacro:property name="steer_joint_damping" value="0.1" />
+  <xacro:property name="steer_joint_friction" value="0.1" />
+  <xacro:property name="steer_joint_effort_limit" value="1000.0" />
+  <xacro:property name="steer_joint_velocity_limit" value="100.0" />
   <xacro:property name="steer_mechanical_reduction" value="1.0" />
   <xacro:property name="steer_joint_position_limit" value="1.56" />
-  <xacro:property name="traction_joint_damping" value="1000.0" />
-  <xacro:property name="traction_joint_friction" value="1000.0" />
-  <xacro:property name="traction_joint_effort_limit" value="100000.0" />
-  <xacro:property name="traction_joint_velocity_limit" value="6.28" />
+  <xacro:property name="traction_joint_damping" value="1.0" />
+  <xacro:property name="traction_joint_friction" value="1.0" />
+  <xacro:property name="traction_joint_effort_limit" value="10.0" />
+  <xacro:property name="traction_joint_velocity_limit" value="10.0" />
   <xacro:property name="traction_mechanical_reduction" value="1.0" />
   <xacro:property name="traction_joint_position_limit" value="1000.0" />
-  <!--xacro:property name="traction_joint_position_limit" value="1000.0" /-->
   <xacro:macro name="cylinder_inertia" params="m r h">
     <inertia ixx="${m*(3*r*r+h*h)/12}" ixy = "0" ixz = "0" iyy="${m*(3*r*r+h*h)/12}" iyz = "0" izz="${m*r*r/2}" />
@@ -28,7 +27,7 @@
       <parent link="${parent}"/>
       <child link="${prefix}wheel_steer_link"/>
-      <xacro:insert_block name="origin" />
-      <axis xyz="0 0 1" rpy="0 0 0" />
-      <limit effort="${steer_joint_effort_limit}" velocity="${steer_joint_velocity_limit}" lower="-${steer_joint_position_limit}" upper="${steer_joint_position_limit}"/>/>
+      <xacro:insert_block name="origin"/>
+      <axis xyz="0 0 1" rpy="0 0 0"/>
+      <limit effort="${steer_joint_effort_limit}" velocity="${steer_joint_velocity_limit}" lower="-${steer_joint_position_limit}" upper="${steer_joint_position_limit}"/>
       <dynamics damping="${steer_joint_damping}" friction="${steer_joint_friction}"/>
     </joint>
@@ -45,17 +44,14 @@
     <link name="${prefix}wheel_steer_link">
       <inertial>
-        <mass value="${wheel_mass}" />
-        <origin xyz="0 0 0" />
-        <cylinder_inertia m="${wheel_mass}" r="${wheel_height}" h="${wheel_radius}" />
+        <mass value="1" />
+        <origin xyz="0 0 -${wheel_radius}" />
+        <cylinder_inertia m="${1}" r="${0.1}" h="${0.1}" />
       </inertial>
     </link>
     <gazebo reference="${prefix}wheel_steer_link">
 			<kp>500000.0</kp>
-			<kd>10.0</kd>
-			<mu1>10</mu1>
-			<mu2>10</mu2>
-			<fdir1>1 0 0</fdir1>
-			<maxVel>1.0</maxVel>
-			<minDepth>0.003</minDepth>
+			<kd>100000.0</kd>
+			<mu1>0</mu1>
+			<mu2>0</mu2>
 			<material>Gazebo/Yellow</material>
 			<turnGravityOff>false</turnGravityOff>
@@ -67,7 +63,7 @@
       <child link="${prefix}wheel_traction_link"/>
       <!--origin xyz="0.1 0 -${wheel_radius}" rpy="0 0 ${M_PI}" /-->
-      <origin xyz="0 0 -${wheel_radius}" rpy="0 0 ${M_PI}" />
-      <axis xyz="0 1 0" rpy="0 0 0" />
-      <limit effort="${traction_joint_effort_limit}" velocity="${traction_joint_velocity_limit}" />
+      <origin xyz="0 0 -${wheel_radius}" rpy="0 0 ${M_PI}"/>
+      <axis xyz="0 1 0" rpy="0 0 0"/>
+      <limit effort="${traction_joint_effort_limit}" velocity="${traction_joint_velocity_limit}"/>
       <dynamics damping="${traction_joint_damping}" friction="${traction_joint_friction}"/>
     </joint>
@@ -98,5 +94,5 @@
       </visual>
       <collision>
-        <origin xyz="0 0 0" rpy="${M_PI/2} 0 0" />
+        <origin xyz="0 0 0" rpy="${M_PI/2} 0 0"/>
         <geometry>
           <cylinder radius="${wheel_radius}" length="${wheel_height}"/>
@@ -110,10 +106,10 @@
     </link>
 		<gazebo reference="${prefix}wheel_traction_link">
-			<kp>500000.0</kp>
-			<kd>5.0</kd>
-			<mu1>18</mu1>
-			<mu2>18</mu2>
+			<kp>5000000</kp>
+			<kd>5000000</kd>
+			<mu1>2</mu1>
+			<mu2>2</mu2>
 			<fdir1>1 0 0</fdir1>
-			<maxVel>1.0</maxVel>
+			<maxVel>3.0</maxVel>
 			<minDepth>0.003</minDepth>
 			<material>Gazebo/Yellow</material>
