Commit message: Fixed an issue with fork_support_wheels. SteeringController is Position/Position ElevatorController is Velocity/Velocity Visual helper wheels is activated

File: hr_recycler_common/hr_recycler_description/robots/hr_recycler_std.urdf.xacro (robot description, xacro)
@@ -79,9 +79,4 @@
       <origin xyz="${camera_x} ${camera_y} ${camera_z}" rpy="0 0 ${PI}"/>
   </xacro:sensor_r430>
-  <!--gazebo>
-    <plugin name="gazebo_ros_control" filename="libgazebo_ros_control.so">
-      <robotSimType>steer_bot_hardware_gazebo/SteerBotHardwareGazebo</robotSimType>
-    </plugin>
-  </gazebo-->
 	<!-- Gazebo ros control pluggins -->
 	<xacro:ros_control/>

File: hr_recycler_common/hr_recycler_description/urdf/bases/hr_recycler.urdf.xacro (robot description, xacro)
@@ -61,12 +61,23 @@
   </link>
   <!-- BASE HELPER! -->
-  <!-- Two small boxes that help the to not tip over -->
+  <!-- Two small spheres that help the to not tip over -->
   <joint name="${prefix}base_helper_joint" type="continuous">
-    <origin xyz="-${base_length/2.0+0.3} ${base_width/2.0-wheel_radius/2.0} -${wheel_radius/2.0}" rpy="0 0 0" />
+    <origin xyz="-${base_length/2.0+0.5} ${base_width/2.0-wheel_radius/2.0} -${wheel_radius/2.0}" rpy="0 0 0" />
     <parent link="${prefix}base_link"/>
     <child link="${prefix}base_helper_link" />
+    <axis xyz="1 0 0" rpy="0 0 0" />
   </joint>
+  <!--transmission name="${prefix}base_helper_joint_trans">
+    <type>transmission_interface/SimpleTransmission</type>
+    <joint name="${prefix}base_helper_joint">
+      <hardwareInterface>hardware_interface/VelocityJointInterface</hardwareInterface>
+    </joint>
+    <actuator name="${prefix}base_helper_joint_motor">
+      <hardwareInterface>hardware_interface/VelocityActuatorInterface</hardwareInterface>
+      <mechanicalReduction>${steer_mechanical_reduction}</mechanicalReduction>
+    </actuator>
+  </transmission-->
   <link name="${prefix}base_helper_link">
-    <!--visual>
+    <visual>
       <origin xyz="0 0 0" rpy="0 0 0" />
       <geometry>
@@ -76,27 +87,43 @@
          <color rgba="0.1 0.1 0.1 1"/>
        </material>
-    </visual-->
-    <collision>
+     </visual>
+     <collision>
       <origin xyz="0 0 0" rpy="0 0 0" />
       <geometry>
         <sphere radius="${wheel_radius/2.0}"/>
       </geometry>
-    </collision>
+      </collision>
+      <inertial>
+        <mass value="${base_mass}" />
+        <origin xyz="0 0 0" />
+        <box_inertia  m="${base_mass}" x="${base_length}" y="${base_width}" z="${base_height}"/>
+      </inertial>
     </link>
     <joint name="${prefix}base_helper_2_joint" type="continuous">
-      <origin xyz="-${base_length/2.0+0.3} -${base_width/2.0-wheel_radius/2.0} -${wheel_radius/2.0}" rpy="0 0 0" />
+      <origin xyz="-${base_length/2.0+0.5} -${base_width/2.0-wheel_radius/2.0} -${wheel_radius/2.0}" rpy="0 0 0" />
       <parent link="${prefix}base_link"/>
       <child link="${prefix}base_helper_2_link" />
+      <axis xyz="1 0 0" rpy="0 0 0" />
     </joint>
+    <!--transmission name="${prefix}base_helper_2_joint_trans">
+      <type>transmission_interface/SimpleTransmission</type>
+      <joint name="${prefix}base_helper_2_joint">
+        <hardwareInterface>hardware_interface/VelocityJointInterface</hardwareInterface>
+      </joint>
+      <actuator name="${prefix}base_helper_2_joint_motor">
+        <hardwareInterface>hardware_interface/VelocityActuatorInterface</hardwareInterface>
+        <mechanicalReduction>${steer_mechanical_reduction}</mechanicalReduction>
+      </actuator>
+    </transmission-->
     <link name="${prefix}base_helper_2_link">
-      <!--visual>
+      <visual>
         <origin xyz="0 0 0" rpy="0 0 0" />
         <geometry>
-           <box size="${wheel_radius} ${wheel_radius} ${wheel_radius}"/>
+          <sphere radius="${wheel_radius/2.0}"/>
         </geometry>
          <material name="darkgrey">
            <color rgba="0.1 0.1 0.1 1"/>
          </material>
-      </visual-->
+      </visual>
       <collision>
         <origin xyz="0 0 0" rpy="0 0 0" />
@@ -105,5 +132,10 @@
         </geometry>
       </collision>
-      </link>
+      <inertial>
+        <mass value="${base_mass}" />
+        <origin xyz="0 0 0" />
+        <box_inertia  m="${base_mass}" x="${base_length}" y="${base_width}" z="${base_height}"/>
+      </inertial>
+    </link>
   </xacro:macro>
 </robot>

File: hr_recycler_common/hr_recycler_description/urdf/common.gazebo.xacro (robot description, xacro)
@@ -9,6 +9,12 @@
         <controlPeriod>0.001</controlPeriod>
 	    <robotSimType>gazebo_ros_control/DefaultRobotHWSim</robotSimType>
+			<legacyModeNS>true</legacyModeNS>
       </plugin>
    </gazebo>
+	   <!--gazebo>
+	     <plugin name="gazebo_ros_control" filename="libgazebo_ros_control.so">
+	       <robotSimType>steer_bot_hardware_gazebo/SteerBotHardwareGazebo</robotSimType>
+	     </plugin>
+	   </gazebo-->
    </xacro:macro>
    <xacro:macro name="gazebo_colors" params="prefix">
@@ -19,4 +25,22 @@
 			<material>Gazebo/Grey</material>
 		</gazebo>
+		<!--gazebo reference="${prefix}base_helper_wheel_link">
+			<mu1 value="5.0"/>
+			<mu2 value="0.5"/>
+			<kp value="10000000.0" />
+			<kd value="1.0" />
+			<fdir1 value="1 0 0"/>
+			<material>Gazebo/Grey</material>
+			<turnGravityOff>false</turnGravityOff>
+		</gazebo-->
+		<!--gazebo reference="${prefix}base_helper_link_2_link">
+			<mu1 value="5.0"/>
+			<mu2 value="0.5"/>
+			<kp value="10000000.0" />
+			<kd value="1.0" />
+			<fdir1 value="1 0 0"/>
+			<material>Gazebo/Grey</material>
+			<turnGravityOff>false</turnGravityOff>
+		</gazebo-->
 		<gazebo reference="$(arg prefix)front_cover_link">
 			<material>Gazebo/Black</material>

File: hr_recycler_common/hr_recycler_description/urdf/elevator/both_elevator.urdf.xacro (robot description, xacro)
@@ -17,11 +17,11 @@
         <limit effort="1000.0" lower="0.0" upper="0.25" velocity="1.0"/>
     </joint>
-    <transmission name="${prefix}both_elevator_transmission">
+    <transmission name="${prefix}_both_elevator_transmission">
       <type>transmission_interface/SimpleTransmission</type>
       <joint name="${prefix}_both_elevator_joint">
-        <hardwareInterface>hardware_interface/PositionJointInterface</hardwareInterface>
+        <hardwareInterface>hardware_interface/VelocityJointInterface</hardwareInterface>
       </joint>
       <actuator name="${prefix}_both_elevator_motor">
-        <hardwareInterface>hardware_interface/PositionActuatorInterface</hardwareInterface>
+        <hardwareInterface>hardware_interface/VelocityActuatorInterface</hardwareInterface>
         <mechanicalReduction>${traction_mechanical_reduction}</mechanicalReduction>
       </actuator>

File: hr_recycler_common/hr_recycler_description/urdf/elevator/elevator.gazebo.xacro (robot description, xacro)
@@ -25,5 +25,5 @@
 			<turnGravityOff>false</turnGravityOff-->
 		</gazebo>
-		<!--gazebo reference="${name}_wheel_link">
+		<gazebo reference="${name}_wheel_link">
 			<kp>500000.0</kp>
 			<kd>10.0</kd>
@@ -36,5 +36,5 @@
 			<turnGravityOff>false</turnGravityOff>
 			<implicitSpringDamper>1</implicitSpringDamper>
-		</gazebo-->
+		</gazebo>
 	</xacro:macro>
 </robot>

File: hr_recycler_common/hr_recycler_description/urdf/elevator/elevator.urdf.xacro (robot description, xacro)
@@ -1,5 +1,4 @@
 <?xml version="1.0"?>
 <robot xmlns:xacro="http://www.ros.org/wiki/xacro">
-	<xacro:include filename="$(find hr_recycler_description)/urdf/elevator/elevator.transmission.xacro"/>
 	<xacro:include filename="$(find hr_recycler_description)/urdf/elevator/elevator.gazebo.xacro"/>
 	<xacro:macro name="elevator_platform" params="prefix parent hq *origin">
@@ -67,13 +66,23 @@
 	</link>
 	<joint name="${prefix}_support_wheel_joint" type="continuous">
-			<origin xyz="${support_wheel_joint_x} ${support_wheel_joint_y} ${support_wheel_joint_z}" rpy="0 0 0"/>
+			<origin xyz="${support_wheel_joint_x} ${support_wheel_joint_y} ${support_wheel_joint_z+0.005}" rpy="0 0 0"/>
 			<parent link="${prefix}_platform_link"/>
 			<child link="${prefix}_support_wheel_link" />
-			<limit effort="1000.0" velocity="1.0"/>
+			<limit effort="1000.0" velocity="100.0"/>
 			<axis xyz="0 1 0" rpy="0 0 0" />
 	</joint>
+	<transmission name="${prefix}_support_wheel_joint_transmission">
+		<type>transmission_interface/SimpleTransmission</type>
+		<joint name="${prefix}_support_wheel_joint">
+			<hardwareInterface>hardware_interface/VelocityJointInterface</hardwareInterface>
+		</joint>
+		<actuator name="${prefix}_both_elevator_motor">
+			<hardwareInterface>hardware_interface/VelocityActuatorInterface</hardwareInterface>
+			<mechanicalReduction>${traction_mechanical_reduction}</mechanicalReduction>
+		</actuator>
+	</transmission>
 	<link name="${prefix}_support_wheel_link">
 		<visual>
-				<origin xyz="0 0 0.01" rpy="${M_PI/2} 0 0" />
+				<origin xyz="0 0 0" rpy="${M_PI/2} 0 0" />
 				<geometry>
 					<cylinder radius="${support_wheel_radius}" length="${support_wheel_length}"/>
@@ -81,5 +90,5 @@
 		</visual>
 		<collision>
-			<origin xyz="0 0 +0.01" rpy="${M_PI/2} 0 0" />
+			<origin xyz="0 0 0" rpy="${M_PI/2} 0 0" />
 			<geometry>
 				<cylinder radius="${support_wheel_radius}" length="${support_wheel_length}"/>

File: hr_recycler_common/hr_recycler_description/urdf/wheels/motor_wheel.urdf.xacro (robot description, xacro)
@@ -10,5 +10,5 @@
   <xacro:property name="steer_joint_friction" value="1000.0" />
   <xacro:property name="steer_joint_effort_limit" value="9999.0" />
-  <xacro:property name="steer_joint_velocity_limit" value="2" />
+  <xacro:property name="steer_joint_velocity_limit" value="200" />
   <xacro:property name="steer_mechanical_reduction" value="1.0" />
   <xacro:property name="steer_joint_position_limit" value="1.56" />
