Commit message: Added Gazebo references and a new system for the elevator.

File: hr_recycler_common/hr_recycler_description/robots/hr_recycler_std.urdf.xacro (robot description, xacro)
@@ -31,8 +31,4 @@
   <xacro:property name="base_height" value="0.533" />
   <xacro:property name="base_width" value="0.754" />
-	<!-- Castor paramters -->
-	<!--xacro:property name="omni_x" value="0.296"/>
-	<xacro:property name="omni_y" value="0.249"/>
-	<xacro:property name="omni_z" value="0.010"/-->
 	<!-- Flag to select the high or low quality model -->
 	<xacro:property name="hq" value="true" />
@@ -55,6 +51,7 @@
 	<xacro:property name="elevator_x" value="-${base_length/2.0}" />
 	<xacro:property name="elevator_y" value="0.0" />
-	<xacro:property name="elevator_z" value="0.0" />
+	<xacro:property name="elevator_z" value="${-wheel_radius/2.0+fork_height/2.0}" />
   <xacro:property name="fork_length" value="1.176" />
+  <xacro:property name="fork_height" value="0.015" />
 	<!-- *************** -->
 	<!-- Robots Elements -->
@@ -80,4 +77,11 @@
   </xacro:sensor_r430>
 	<!-- Gazebo ros control pluggins -->
+  <gazebo>
+    <plugin name="gazebo_ros_control" filename="libgazebo_ros_control.so">
+      <robotNamespace>/hr_recycler</robotNamespace>
+      <robotSimType>gazebo_ros_control/DefaultRobotHWSim</robotSimType>
+      <legacyModeNS>true</legacyModeNS>
+    </plugin>
+  </gazebo>
 	<xacro:ros_control/>
 </robot>

File: hr_recycler_common/hr_recycler_description/urdf/bases/hr_recycler.urdf.xacro (robot description, xacro)
@@ -9,5 +9,5 @@
   <xacro:property name="base_width" value="0.754" />
   <xacro:property name="base_height" value="0.533" />
-  <xacro:property name="base_mass" value="25.0"/>
+  <xacro:property name="base_mass" value="50.0"/>
   <xacro:property name="visual_base_link_z" value="${wheel_radius+base_height/2.0+separation_wheel_box}" />
   <xacro:property name="fork_length" value="1.176" />
@@ -22,5 +22,4 @@
   </xacro:macro>
   <!-- BASE FOOTPRINT -->
-  <xacro:if value="${publish_bf}">
     <link name="${prefix}base_footprint">
       <visual>
@@ -36,5 +35,4 @@
       <child link="${prefix}base_link" />
     </joint>
-  </xacro:if>
   <!-- BASE_LINK -->
   <link name="${prefix}base_link">
@@ -60,82 +58,4 @@
     </collision>
   </link>
-  <!-- BASE HELPER! -->
-  <!-- Two small spheres that help the to not tip over -->
-  <joint name="${prefix}base_helper_joint" type="continuous">
-    <origin xyz="-${base_length/2.0+0.5} ${base_width/2.0-wheel_radius/2.0} -${wheel_radius/2.0}" rpy="0 0 0" />
-    <parent link="${prefix}base_link"/>
-    <child link="${prefix}base_helper_link" />
-    <axis xyz="1 0 0" rpy="0 0 0" />
-  </joint>
-  <!--transmission name="${prefix}base_helper_joint_trans">
-    <type>transmission_interface/SimpleTransmission</type>
-    <joint name="${prefix}base_helper_joint">
-      <hardwareInterface>hardware_interface/VelocityJointInterface</hardwareInterface>
-    </joint>
-    <actuator name="${prefix}base_helper_joint_motor">
-      <hardwareInterface>hardware_interface/VelocityActuatorInterface</hardwareInterface>
-      <mechanicalReduction>${steer_mechanical_reduction}</mechanicalReduction>
-    </actuator>
-  </transmission-->
-  <link name="${prefix}base_helper_link">
-    <visual>
-      <origin xyz="0 0 0" rpy="0 0 0" />
-      <geometry>
-         <sphere radius="${wheel_radius/2.0}"/>
-      </geometry>
-       <material name="darkgrey">
-         <color rgba="0.1 0.1 0.1 1"/>
-       </material>
-     </visual>
-     <collision>
-      <origin xyz="0 0 0" rpy="0 0 0" />
-      <geometry>
-        <sphere radius="${wheel_radius/2.0}"/>
-      </geometry>
-      </collision>
-      <inertial>
-        <mass value="${base_mass}" />
-        <origin xyz="0 0 0" />
-        <box_inertia  m="${base_mass}" x="${base_length}" y="${base_width}" z="${base_height}"/>
-      </inertial>
-    </link>
-    <joint name="${prefix}base_helper_2_joint" type="continuous">
-      <origin xyz="-${base_length/2.0+0.5} -${base_width/2.0-wheel_radius/2.0} -${wheel_radius/2.0}" rpy="0 0 0" />
-      <parent link="${prefix}base_link"/>
-      <child link="${prefix}base_helper_2_link" />
-      <axis xyz="1 0 0" rpy="0 0 0" />
-    </joint>
-    <!--transmission name="${prefix}base_helper_2_joint_trans">
-      <type>transmission_interface/SimpleTransmission</type>
-      <joint name="${prefix}base_helper_2_joint">
-        <hardwareInterface>hardware_interface/VelocityJointInterface</hardwareInterface>
-      </joint>
-      <actuator name="${prefix}base_helper_2_joint_motor">
-        <hardwareInterface>hardware_interface/VelocityActuatorInterface</hardwareInterface>
-        <mechanicalReduction>${steer_mechanical_reduction}</mechanicalReduction>
-      </actuator>
-    </transmission-->
-    <link name="${prefix}base_helper_2_link">
-      <visual>
-        <origin xyz="0 0 0" rpy="0 0 0" />
-        <geometry>
-          <sphere radius="${wheel_radius/2.0}"/>
-        </geometry>
-         <material name="darkgrey">
-           <color rgba="0.1 0.1 0.1 1"/>
-         </material>
-      </visual>
-      <collision>
-        <origin xyz="0 0 0" rpy="0 0 0" />
-        <geometry>
-          <sphere radius="${wheel_radius/2.0}"/>
-        </geometry>
-      </collision>
-      <inertial>
-        <mass value="${base_mass}" />
-        <origin xyz="0 0 0" />
-        <box_inertia  m="${base_mass}" x="${base_length}" y="${base_width}" z="${base_height}"/>
-      </inertial>
-    </link>
   </xacro:macro>
 </robot>

File: hr_recycler_common/hr_recycler_description/urdf/elevator/both_elevator.urdf.xacro (robot description, xacro)
@@ -3,28 +3,20 @@
   <xacro:include filename="$(find hr_recycler_description)/urdf/elevator/elevator.urdf.xacro"/>
   <xacro:macro name="both_elevator" params="prefix parent hq *origin" >
+    <xacro:property name="elevator_x" value="0.0" />
+  	<xacro:property name="elevator_y" value="0.195" />
+  	<xacro:property name="elevator_z" value="${fork_height}" />
     <xacro:property name="fork_length" value="1.176" />
-    <xacro:property name="elevator_x" value="-${base_length/2.0}" />
-  	<xacro:property name="elevator_y" value="0.195" />
-  	<xacro:property name="elevator_z" value="0.0" />
   	<xacro:property name="fork_width" value="0.11" />
-  	<xacro:property name="fork_height" value="0.05" />
+  	<xacro:property name="fork_height" value="0.015" />
   	<xacro:property name="fork_mass" value="10.0" />
-    <joint name="${prefix}_both_elevator_joint" type="prismatic">
+    <xacro:property name="fork_separation" value="0.116" />
+    <xacro:property name="fork_x" value="0.0" />
+    <xacro:property name="fork_y" value="0.195" />
+    <xacro:property name="fork_z" value="0.0" />
+    <joint name="${prefix}_both_elevator_joint" type="fixed">
         <xacro:insert_block name="origin" />
         <parent link="${parent}"/>
         <child link="${prefix}_platform_link" />
-        <axis xyz="0 0 1"/>
-        <limit effort="1000.0" lower="0.0" upper="0.25" velocity="1.0"/>
     </joint>
-    <transmission name="${prefix}_both_elevator_transmission">
-      <type>transmission_interface/SimpleTransmission</type>
-      <joint name="${prefix}_both_elevator_joint">
-        <hardwareInterface>hardware_interface/VelocityJointInterface</hardwareInterface>
-      </joint>
-      <actuator name="${prefix}_both_elevator_motor">
-        <hardwareInterface>hardware_interface/VelocityActuatorInterface</hardwareInterface>
-        <mechanicalReduction>${traction_mechanical_reduction}</mechanicalReduction>
-      </actuator>
-    </transmission>
     <link name="${prefix}_platform_link">
       <inertial>
@@ -35,9 +27,105 @@
     </link>
     <xacro:elevator_platform prefix="$(arg prefix)left_fork" parent="${prefix}_platform_link" hq="${hq}">
-        <origin xyz="0 ${elevator_y} -0.02" rpy="0 0 0"/>
+        <origin xyz="${fork_x} ${fork_y} ${fork_z}" rpy="0 0 0"/>
     </xacro:elevator_platform>
     <xacro:elevator_platform prefix="$(arg prefix)right_fork" parent="${prefix}_platform_link" hq="${hq}">
-        <origin xyz="0 -${elevator_y} -0.02" rpy="0 0 0"/>
+        <origin xyz="${fork_x} -${fork_y} ${fork_z}" rpy="0 0 0"/>
     </xacro:elevator_platform>
+    <joint name="${prefix}_prismatic_both_forks_joint" type="prismatic">
+        <origin xyz="0 0 0" rpy="0 0 0"/>
+        <parent link="${prefix}_platform_link"/>
+        <child link="${prefix}_prismatic_forks_link" />
+        <axis xyz="0 0 1"/>
+        <limit effort="1000.0" lower="0.0" upper="0.25" velocity="1"/>
+    </joint>
+    <transmission name="${prefix}_prismatic_both_forks_joint_transmission">
+      <type>transmission_interface/SimpleTransmission</type>
+      <joint name="${prefix}_prismatic_both_forks_joint">
+        <hardwareInterface>hardware_interface/PositionJointInterface</hardwareInterface>
+      </joint>
+      <actuator name="${prefix}_prismatic_both_forks_joint_motor">
+        <hardwareInterface>hardware_interface/PositionActuatorInterface</hardwareInterface>
+        <mechanicalReduction>${traction_mechanical_reduction}</mechanicalReduction>
+      </actuator>
+    </transmission>
+    <link name="${prefix}_prismatic_forks_link">
+      <inertial>
+        <mass value="${fork_mass}" />
+        <origin xyz="0 0 1" />
+        <solid_cuboid_inertia m="${fork_mass/2.0}" h="${fork_height}" d="${fork_length}" w="${fork_width}"/>
+      </inertial>
+    </link>
+    <joint name="${prefix}_prismatic_left_fork_joint" type="fixed">
+        <origin xyz="${elevator_x} ${elevator_y} ${elevator_z}" rpy="0 0 0"/>
+        <parent link="${prefix}_prismatic_forks_link"/>
+        <child link="${prefix}_prismatic_left_fork" />
+    </joint>
+    <link name="${prefix}_prismatic_left_fork">
+      <visual>
+        <origin xyz="-${fork_length/2} 0 0" rpy="0 0 0" />
+        <xacro:if value="${hq}">
+          <geometry>
+            <!--mesh filename="package://hr_recycler_description/meshes/elevator/hr_recycler_elevator.dae"/-->
+            <box size="${fork_length} ${fork_width} ${fork_height}"/>
+          </geometry>
+        </xacro:if>
+        <xacro:unless value="${hq}">
+          <geometry>
+            <!--mesh filename="package://hr_recycler_description/meshes/elevator/hr_recycler_elevator.stl"/-->
+            <box size="${fork_length} ${fork_width} ${fork_height}"/>
+          </geometry>
+        </xacro:unless>
+        <material name="black">
+          <color rgba="0.0 0.0 0.0 1"/>
+        </material>
+      </visual>
+      <collision>
+        <origin xyz="-${fork_length/2} 0 0" rpy="0 0 0" />
+        <geometry>
+          <box size="${fork_length} ${fork_width} ${fork_height}"/>
+        </geometry>
+      </collision>
+      <inertial>
+        <mass value="${fork_mass}" />
+        <origin xyz="-1 0 0" />
+        <solid_cuboid_inertia m="${fork_mass}" h="${fork_height}" d="${fork_length}" w="${fork_width}"/>
+      </inertial>
+    </link>
+    <joint name="${prefix}_prismatic_right_fork_joint" type="fixed">
+        <origin xyz="${elevator_x} -${elevator_y} ${elevator_z}" rpy="0 0 0"/>
+        <parent link="${prefix}_prismatic_forks_link"/>
+        <child link="${prefix}_prismatic_right_fork" />
+    </joint>
+    <link name="${prefix}_prismatic_right_fork">
+      <visual>
+        <origin xyz="-${fork_length/2} 0 0" rpy="0 0 0" />
+        <xacro:if value="${hq}">
+          <geometry>
+            <!--mesh filename="package://hr_recycler_description/meshes/elevator/hr_recycler_elevator.dae"/-->
+            <box size="${fork_length} ${fork_width} ${fork_height}"/>
+          </geometry>
+        </xacro:if>
+        <xacro:unless value="${hq}">
+          <geometry>
+            <!--mesh filename="package://hr_recycler_description/meshes/elevator/hr_recycler_elevator.stl"/-->
+            <box size="${fork_length} ${fork_width} ${fork_height}"/>
+          </geometry>
+        </xacro:unless>
+        <material name="black">
+          <color rgba="0.0 0.0 0.0 1"/>
+        </material>
+      </visual>
+      <collision>
+        <origin xyz="-${fork_length/2} 0 0" rpy="0 0 0" />
+        <geometry>
+          <box size="${fork_length} ${fork_width} ${fork_height}"/>
+        </geometry>
+      </collision>
+      <inertial>
+        <mass value="${fork_mass}" />
+        <origin xyz="-1 0 0" />
+        <solid_cuboid_inertia m="${fork_mass}" h="${fork_height}" d="${fork_length}" w="${fork_width}"/>
+      </inertial>
+    </link>
   </xacro:macro>
 </robot>

File: hr_recycler_common/hr_recycler_description/urdf/elevator/elevator.gazebo.xacro (robot description, xacro)
@@ -10,9 +10,9 @@
 			<material>Gazebo/Grey</material>
 			<turnGravityOff>false</turnGravityOff>
-			<!--kp>500000.0</kp>
+			<kp>500000.0</kp>
 			<kd>10.0</kd>
 			<mu1>10</mu1>
 			<mu2>10</mu2>
-			<fdir1>1 0 0</fdir1-->
+			<fdir1>1 0 0</fdir1>
 			<!--minDepth>0.001</minDepth-->
 			<!--material>Gazebo/Black</material-->
@@ -25,15 +25,26 @@
 			<turnGravityOff>false</turnGravityOff-->
 		</gazebo>
-		<gazebo reference="${name}_wheel_link">
+		<gazebo reference="${prefix}_support_wheel_link">
+			<mu1 value="5.0"/>
+			<mu2 value="0.5"/>
+			<kp value="10000000.0" />
+			<kd value="1.0" />
+			<fdir1 value="1 0 0"/>
+			<material>Gazebo/Grey</material>
+			<turnGravityOff>false</turnGravityOff>
 			<kp>500000.0</kp>
 			<kd>10.0</kd>
-			<mu1>10</mu1>
-			<mu2>10</mu2>
+			<mu1>0.2</mu1>
+			<mu2>0.2</mu2>
 			<fdir1>1 0 0</fdir1>
-			<maxVel>1.0</maxVel>
-			<minDepth>0.003</minDepth>
+			<!--minDepth>0.001</minDepth-->
+			<!--material>Gazebo/Black</material-->
+			<!--mu1 value="10"/>
+			<mu2 value="5"/>
+			<kp value="500000.0" />
+			<kd value="10.0" />
+			<fdir1 value="1 0 0"/>
 			<material>Gazebo/Yellow</material>
-			<turnGravityOff>false</turnGravityOff>
-			<implicitSpringDamper>1</implicitSpringDamper>
+			<turnGravityOff>false</turnGravityOff-->
 		</gazebo>
 	</xacro:macro>

File: hr_recycler_common/hr_recycler_description/urdf/elevator/elevator.urdf.xacro (robot description, xacro)
@@ -5,13 +5,13 @@
 	<xacro:property name="fork_length" value="1.176" />
 	<xacro:property name="fork_width" value="0.11" />
-	<xacro:property name="fork_height" value="0.03" />
-	<xacro:property name="fork_mass" value="25.0" />
+	<xacro:property name="fork_height" value="0.015" />
+	<xacro:property name="fork_mass" value="10.0" />
 	<xacro:property name="fork_separation" value="0.116" />
-	<xacro:property name="support_wheel_radius" value="${wheel_radius/2.0-fork_height/2.0}" />
+	<xacro:property name="support_wheel_radius" value="${wheel_radius/4.0}" />
 	<xacro:property name="support_wheel_length" value="${fork_width}" />
-  <xacro:property name="support_wheel_mass" value="5.0" />
+  <xacro:property name="support_wheel_mass" value="10.0" />
 	<xacro:property name="support_wheel_joint_x" value="${0.16-fork_length}" />
 	<xacro:property name="support_wheel_joint_y" value="0.0" />
-	<xacro:property name="support_wheel_joint_z" value="-${wheel_radius/2.0+fork_height/4.0}" />
+	<xacro:property name="support_wheel_joint_z" value="-${fork_height/2.0+support_wheel_radius}" />
 	<!-- PARAMS: -->
 	<!-- name : name of the link: -->
@@ -61,23 +61,23 @@
 		<inertial>
 			<mass value="${fork_mass}" />
-			<origin xyz="0 0 -0.27" />
+			<origin xyz="-${fork_length} 0 0" />
 			<solid_cuboid_inertia m="${fork_mass}" h="${fork_height}" d="${fork_length}" w="${fork_width}"/>
 		</inertial>
 	</link>
 	<joint name="${prefix}_support_wheel_joint" type="continuous">
-			<origin xyz="${support_wheel_joint_x} ${support_wheel_joint_y} ${support_wheel_joint_z+0.005}" rpy="0 0 0"/>
+			<origin xyz="${support_wheel_joint_x} ${support_wheel_joint_y} ${support_wheel_joint_z}" rpy="0 0 0"/>
 			<parent link="${prefix}_platform_link"/>
 			<child link="${prefix}_support_wheel_link" />
 			<limit effort="1000.0" velocity="100.0"/>
-			<axis xyz="0 1 0" rpy="0 0 0" />
+			<axis xyz="0 -1 0" rpy="0 0 0" />
 	</joint>
-	<transmission name="${prefix}_support_wheel_joint_transmission">
-		<type>transmission_interface/SimpleTransmission</type>
-		<joint name="${prefix}_support_wheel_joint">
-			<hardwareInterface>hardware_interface/VelocityJointInterface</hardwareInterface>
+  <transmission name="${prefix}_support_wheel_joint_transmission">
+  	<type>transmission_interface/SimpleTransmission</type>
+	  <joint name="${prefix}_support_wheel_joint">
+    	<hardwareInterface>hardware_interface/VelocityJointInterface</hardwareInterface>
 		</joint>
 		<actuator name="${prefix}_both_elevator_motor">
 			<hardwareInterface>hardware_interface/VelocityActuatorInterface</hardwareInterface>
-			<mechanicalReduction>${traction_mechanical_reduction}</mechanicalReduction>
+			<mechanicalReduction>$1</mechanicalReduction>
 		</actuator>
 	</transmission>
@@ -101,4 +101,9 @@
 		</inertial>
 	</link>
+	<gazebo reference="${prefix}_support_wheel_link">
+    <mu1>10</mu1>
+    <mu2>10</mu2>
+    <material>Gazebo/Black</material>
+  </gazebo>
 	<!--xacro:elevator_transmission prefix="${prefix}" /-->
 	<!--xacro:elevator_gazebo prefix="${prefix}" /-->

File: hr_recycler_common/hr_recycler_description/urdf/wheels/motor_wheel.urdf.xacro (robot description, xacro)
@@ -50,8 +50,21 @@
       </inertial>
     </link>
+    <gazebo reference="${prefix}wheel_steer_link">
+			<kp>500000.0</kp>
+			<kd>10.0</kd>
+			<mu1>10</mu1>
+			<mu2>10</mu2>
+			<fdir1>1 0 0</fdir1>
+			<maxVel>1.0</maxVel>
+			<minDepth>0.003</minDepth>
+			<material>Gazebo/Yellow</material>
+			<turnGravityOff>false</turnGravityOff>
+			<implicitSpringDamper>1</implicitSpringDamper>
+		</gazebo>
     <!--WHEEL TIRE -->
     <joint name="${prefix}wheel_traction_joint" type="continuous">
       <parent link="${prefix}wheel_steer_link"/>
       <child link="${prefix}wheel_traction_link"/>
+      <!--origin xyz="0.1 0 -${wheel_radius}" rpy="0 0 ${M_PI}" /-->
       <origin xyz="0 0 -${wheel_radius}" rpy="0 0 ${M_PI}" />
       <axis xyz="0 1 0" rpy="0 0 0" />
@@ -96,4 +109,16 @@
       </inertial>
     </link>
+		<gazebo reference="${prefix}wheel_traction_link">
+			<kp>500000.0</kp>
+			<kd>5.0</kd>
+			<mu1>18</mu1>
+			<mu2>18</mu2>
+			<fdir1>1 0 0</fdir1>
+			<maxVel>1.0</maxVel>
+			<minDepth>0.003</minDepth>
+			<material>Gazebo/Yellow</material>
+			<turnGravityOff>false</turnGravityOff>
+			<implicitSpringDamper>1</implicitSpringDamper>
+		</gazebo>
   </xacro:macro>
 </robot>
