Commit message: test in melodic

File: hr_recycler_common/hr_recycler_description/robots/hr_recycler_std.urdf.xacro (robot description, xacro)
@@ -66,18 +66,18 @@
 	<xacro:hr_recycler prefix="$(arg prefix)" publish_bf="true" hq="${hq}" />
 	<xacro:motor_wheel prefix="$(arg prefix)back" parent="$(arg prefix)base_link" hq="${hq}">
-			<origin xyz="${wheel_offset_x} ${wheel_offset_y} ${wheel_offset_z}" rpy="0 0 0"/>
+	    <origin xyz="${wheel_offset_x} ${wheel_offset_y} ${wheel_offset_z}" rpy="0 0 0"/>
 	</xacro:motor_wheel>
-  <xacro:both_elevator prefix="$(arg prefix)both_forks" parent="$(arg prefix)base_link" hq="${hq}">
-      <origin xyz="${elevator_x} ${elevator_y} ${elevator_z+0.01}" rpy="0 0 0"/>
-  </xacro:both_elevator>
-  <xacro:sensor_sick_s300 prefix="$(arg prefix)front_laser" parent="$(arg prefix)base_link">
-      <origin xyz="${sensor_x} ${sensor_y} ${sensor_z}" rpy="${PI} 0 0"/>
-  </xacro:sensor_sick_s300>
-  <xacro:sensor_r430 prefix="$(arg prefix)right_fork_camera" parent="$(arg prefix)right_fork_platform_link" prefix_topic="front_right_rgbd_camera">
-      <origin xyz="${camera_x} ${camera_y} ${camera_z}" rpy="0 0 ${PI}"/>
-  </xacro:sensor_r430>
-  <xacro:sensor_r430 prefix="$(arg prefix)left_fork_camera" parent="$(arg prefix)left_fork_platform_link" prefix_topic="front_left_rgbd_camera">
-      <origin xyz="${camera_x} ${camera_y} ${camera_z}" rpy="0 0 ${PI}"/>
-  </xacro:sensor_r430>
+    <xacro:both_elevator prefix="$(arg prefix)both_forks" parent="$(arg prefix)base_link" hq="true">
+        <origin xyz="${elevator_x} ${elevator_y} ${elevator_z+0.01}" rpy="0 0 0"/>
+    </xacro:both_elevator>
+    <!--<xacro:sensor_sick_s300 prefix="$(arg prefix)front_laser" parent="$(arg prefix)base_link">-->
+        <!--<origin xyz="${sensor_x} ${sensor_y} ${sensor_z}" rpy="${PI} 0 0"/>-->
+    <!--</xacro:sensor_sick_s300>-->
+    <!--<xacro:sensor_r430 prefix="$(arg prefix)right_fork_camera" parent="$(arg prefix)right_fork_platform_link" prefix_topic="front_right_rgbd_camera">-->
+        <!--<origin xyz="${camera_x} ${camera_y} ${camera_z}" rpy="0 0 ${PI}"/>-->
+    <!--</xacro:sensor_r430>-->
+    <!--<xacro:sensor_r430 prefix="$(arg prefix)left_fork_camera" parent="$(arg prefix)left_fork_platform_link" prefix_topic="front_left_rgbd_camera">-->
+        <!--<origin xyz="${camera_x} ${camera_y} ${camera_z}" rpy="0 0 ${PI}"/>-->
+    <!--</xacro:sensor_r430>-->
 	<!-- Gazebo ros control pluggins -->
 	<xacro:ros_control/>

File: hr_recycler_common/hr_recycler_description/urdf/bases/hr_recycler.urdf.xacro (robot description, xacro)
@@ -6,8 +6,8 @@
   <xacro:property name="wheel_width" value="0.220" />
   <xacro:property name="wheel_radius" value="0.10" />
-  <xacro:property name="base_length" value="0.679" />
-  <xacro:property name="base_width" value="0.754" />
-  <xacro:property name="base_height" value="0.533" />
-  <xacro:property name="base_mass" value="2"/>
+  <xacro:property name="base_length" value="0.279" />
+  <xacro:property name="base_width" value="0.354" />
+  <xacro:property name="base_height" value="0.233" />
+  <xacro:property name="base_mass" value="200"/>
   <xacro:property name="visual_base_link_z" value="${wheel_radius+base_height/2.0+separation_wheel_box}" />
   <xacro:property name="fork_length" value="1.176" />

File: hr_recycler_common/hr_recycler_description/urdf/elevator/both_elevator.urdf.xacro (robot description, xacro)
@@ -9,5 +9,5 @@
   	<xacro:property name="fork_width" value="0.11" />
   	<xacro:property name="fork_height" value="0.015" />
-  	<xacro:property name="fork_mass" value="1.0" />
+  	<xacro:property name="fork_mass" value="15.0" />
     <xacro:property name="fork_separation" value="0.116" />
     <xacro:property name="fork_x" value="0.0" />

File: hr_recycler_common/hr_recycler_description/urdf/elevator/elevator.urdf.xacro (robot description, xacro)
@@ -6,5 +6,5 @@
 	<xacro:property name="fork_width" value="0.11" />
 	<xacro:property name="fork_height" value="0.015" />
-	<xacro:property name="fork_mass" value="2.0" />
+	<xacro:property name="fork_mass" value="20.0" />
 	<xacro:property name="fork_separation" value="0.116" />
 	<xacro:property name="support_wheel_radius" value="${wheel_radius/4.0}" />

File: hr_recycler_common/hr_recycler_description/urdf/wheels/omni_wheel.urdf.xacro (robot description, xacro)
@@ -42,11 +42,15 @@
       <origin xyz="0 0 0" rpy="${M_PI/2} 0 0" />
       <geometry>
-         <sphere radius="${omni_wheel_radius*0.35}"/>
+         <!--<sphere radius="${omni_wheel_radius*0.35}"/>-->
+            <cylinder length="${omni_wheel_height}" radius="${omni_wheel_radius*0.35}" />
       </geometry>
       <surface>
         <friction>
           <ode>
-            <mu>0.0001</mu>
-            <mu2>0.0001</mu2>
+                <mu>100.000000</mu>
+                <mu2>0.000000</mu2>
+                <!--<fdir1>0.000000 0.000000 0.000000</fdir1>-->
+                <slip1>0.000000</slip1>
+                <slip2>0.000000</slip2>
           </ode>
         </friction>
