Commit message: change laser position

File: pallet_truck_common/pallet_truck_description/robots/pallet_truck_std.urdf.xacro (robot description, xacro)
@@ -31,5 +31,5 @@
  <xacro:property name="front_laser_x" value="0.25294" />
  <xacro:property name="front_laser_y" value="0.000" />
- <xacro:property name="front_laser_z" value="0.200" />
+ <xacro:property name="front_laser_z" value="0.27" />
 	<!-- *************** -->
 	<!-- Robots Elements -->

Commit message: Fixed prefix and added depth camera

File: pallet_truck_common/pallet_truck_description/robots/pallet_truck_std.urdf.xacro (robot description, xacro)
@@ -67,5 +67,5 @@
 	<!-- *************** -->
 	<!-- Here we create the robot elements using the xacro:macros imported at the beggining of this file -->
-	<xacro:arg name="prefix" default="pallet_truck_"/>
+	<xacro:arg name="prefix" default="pallet_truck/"/>
   <xacro:property name="prefix" value="$(arg prefix)" />
 	<xacro:pallet_truck prefix="${prefix}" publish_bf="true"/> <!-- BASE -->
@@ -97,4 +97,10 @@
       <origin xyz="${front_laser_x} ${front_laser_y} ${front_laser_z}" rpy="${PI} 0 0"/>
   </xacro:sensor_sick_s300>
+  <xacro:sensor_r430 prefix="${prefix}camera_left" parent="${prefix}left_fork_wheel_link">
+  	<origin xyz="-0.181 0 0.029" rpy="0 0 ${PI}"/>
+  </xacro:sensor_r430>
+	<xacro:sensor_r430 prefix="${prefix}camera_right" parent="${prefix}right_fork_wheel_link">
+    <origin xyz="-0.181 0 0.029" rpy="0 0 ${PI}"/>
+  </xacro:sensor_r430>
   <!-- REGISTERS -->
   <!-- Front -->

Commit message: Inserted cameras for pallet detection

File: pallet_truck_common/pallet_truck_description/robots/pallet_truck_std.urdf.xacro (robot description, xacro)
@@ -97,4 +97,5 @@
       <origin xyz="${front_laser_x} ${front_laser_y} ${front_laser_z}" rpy="${PI} 0 0"/>
   </xacro:sensor_sick_s300>
+	<!-- Depth cameras inside forks for pallet detection -->
   <xacro:sensor_r430 prefix="${prefix}camera_left" parent="${prefix}left_fork_wheel_link">
   	<origin xyz="-0.181 0 0.029" rpy="0 0 ${PI}"/>
@@ -103,4 +104,11 @@
     <origin xyz="-0.181 0 0.029" rpy="0 0 ${PI}"/>
   </xacro:sensor_r430>
+	<!-- RGB-D camera for human detection -->
+	<!-- <xacro:sensor_r430 prefix="${prefix}camera_front" parent="${prefix}front_register_link">
+    <origin xyz="0.02 0 0" rpy="0 0 0"/>
+  </xacro:sensor_r430> -->
+	<!-- <xacro:sensor_orbbec_astra prefix="${prefix}camera_front" parent="${prefix}front_register_link">
+    <origin xyz="0.02 0 0" rpy="0 0 0"/>
+  </xacro:sensor_orbbec_astra> -->
   <!-- REGISTERS -->
   <!-- Front -->

Commit message: Added camera for human detection

File: pallet_truck_common/pallet_truck_description/robots/pallet_truck_std.urdf.xacro (robot description, xacro)
@@ -110,9 +110,9 @@
 	<!-- RGB-D camera for human detection -->
 	<!-- <xacro:sensor_r430 prefix="${prefix}camera_front" parent="${prefix}front_register_link">
-    <origin xyz="0.02 0 0" rpy="0 0 0"/>
+    <origin xyz="0.02 0 0.08" rpy="0 -0.785398163 0"/>
   </xacro:sensor_r430> -->
-	<!-- <xacro:sensor_orbbec_astra prefix="${prefix}camera_front" parent="${prefix}front_register_link">
-    <origin xyz="0.02 0 0" rpy="0 0 0"/>
-  </xacro:sensor_orbbec_astra> -->
+	<xacro:sensor_r430 prefix="${prefix}camera_front" parent="${prefix}rplidar_laser_base_link">
+    <origin xyz="0.045 0 -0.09" rpy="0 -0.34906585 0"/>
+  </xacro:sensor_r430>
   <!-- REGISTERS -->
   <!-- Front -->

Commit message: Kept a single depth camera in the left fork

File: pallet_truck_common/pallet_truck_description/robots/pallet_truck_std.urdf.xacro (robot description, xacro)
@@ -105,11 +105,8 @@
   	<origin xyz="-0.181 0 0.029" rpy="0 0 ${PI}"/>
   </xacro:sensor_r430>
-	<xacro:sensor_r430 prefix="${prefix}camera_right" parent="${prefix}right_fork_wheel_link">
+	<!-- <xacro:sensor_r430 prefix="${prefix}camera_right" parent="${prefix}right_fork_wheel_link">
     <origin xyz="-0.181 0 0.029" rpy="0 0 ${PI}"/>
-  </xacro:sensor_r430>
+  </xacro:sensor_r430> -->
 	<!-- RGB-D camera for human detection -->
-	<!-- <xacro:sensor_r430 prefix="${prefix}camera_front" parent="${prefix}front_register_link">
-    <origin xyz="0.02 0 0.08" rpy="0 -0.785398163 0"/>
-  </xacro:sensor_r430> -->
 	<xacro:sensor_r430 prefix="${prefix}camera_front" parent="${prefix}rplidar_laser_base_link">
     <origin xyz="0.045 0 -0.09" rpy="0 -0.34906585 0"/>

Commit message: Added camera_id parameter to fix namespaces in topics and tf frames

File: pallet_truck_common/pallet_truck_description/robots/pallet_truck_std.urdf.xacro (robot description, xacro)
@@ -72,5 +72,5 @@
 	<!-- Here we create the robot elements using the xacro:macros imported at the beggining of this file -->
 	<xacro:arg name="prefix" default="pallet_truck/"/>
-  <xacro:property name="prefix" value="$(arg prefix)" />
+  <xacro:property name="prefix" value="$(arg prefix)"/>
 	<xacro:pallet_truck prefix="${prefix}" publish_bf="true"/> <!-- BASE -->
 	<xacro:motor_wheel prefix="${prefix}" parent="${prefix}front_case_link">
@@ -101,13 +101,10 @@
       <origin xyz="${front_laser_x} ${front_laser_y} ${front_laser_z}" rpy="${PI} 0 0"/>
   </xacro:sensor_sick_s300>
-	<!-- Depth cameras inside forks for pallet detection -->
-  <xacro:sensor_r430 prefix="${prefix}camera_left" parent="${prefix}left_fork_wheel_link">
+	<!-- Depth camera inside left fork for pallet detection -->
+  <xacro:sensor_r430 camera_id="camera_rear" prefix="${prefix}camera_rear" parent="${prefix}left_fork_wheel_link">
   	<origin xyz="-0.181 0 0.029" rpy="0 0 ${PI}"/>
   </xacro:sensor_r430>
-	<!-- <xacro:sensor_r430 prefix="${prefix}camera_right" parent="${prefix}right_fork_wheel_link">
-    <origin xyz="-0.181 0 0.029" rpy="0 0 ${PI}"/>
-  </xacro:sensor_r430> -->
 	<!-- RGB-D camera for human detection -->
-	<xacro:sensor_r430 prefix="${prefix}camera_front" parent="${prefix}rplidar_laser_base_link">
+	<xacro:sensor_r430 camera_id="camera_front" prefix="${prefix}camera_front" parent="${prefix}rplidar_laser_base_link">
     <origin xyz="0.045 0 -0.09" rpy="0 -0.34906585 0"/>
   </xacro:sensor_r430>

Commit message: Changed camera prefixes

File: pallet_truck_common/pallet_truck_description/robots/pallet_truck_std.urdf.xacro (robot description, xacro)
@@ -101,11 +101,11 @@
       <origin xyz="${front_laser_x} ${front_laser_y} ${front_laser_z}" rpy="${PI} 0 0"/>
   </xacro:sensor_sick_s300>
-	<!-- Depth camera inside left fork for pallet detection -->
-  <xacro:sensor_r430 camera_id="camera_rear" prefix="${prefix}camera_rear" parent="${prefix}left_fork_wheel_link">
+	<!-- Human tracking camera -->
+	<xacro:sensor_r430 camera_id="front_camera" prefix="${prefix}front_camera" parent="${prefix}rplidar_laser_base_link">
+    <origin xyz="0.045 0 -0.09" rpy="0 -0.34906585 0"/>
+  </xacro:sensor_r430>
+	<!-- Pallet detection camera -->
+  <xacro:sensor_r430 camera_id="rear_camera" prefix="${prefix}rear_camera" parent="${prefix}left_fork_wheel_link">
   	<origin xyz="-0.181 0 0.029" rpy="0 0 ${PI}"/>
-  </xacro:sensor_r430>
-	<!-- RGB-D camera for human detection -->
-	<xacro:sensor_r430 camera_id="camera_front" prefix="${prefix}camera_front" parent="${prefix}rplidar_laser_base_link">
-    <origin xyz="0.045 0 -0.09" rpy="0 -0.34906585 0"/>
   </xacro:sensor_r430>
   <!-- REGISTERS -->

Commit message: Changed fork camera angle to work with pallet detection method

File: pallet_truck_common/pallet_truck_description/robots/pallet_truck_std.urdf.xacro (robot description, xacro)
@@ -103,12 +103,12 @@
       <origin xyz="${front_support_wheel_offset_x} -${front_support_wheel_offset_y} ${front_support_wheel_offset_z}" rpy="0 0 0"/>
   </xacro:support_wheel>
-  <xacro:sensor_rslidar_16 prefix="${prefix}top_lidar" parent="${prefix}front_case_link" prefix_topic="top_lidar" gpu="${gpu}">
+  <!-- <xacro:sensor_rslidar_16 prefix="${prefix}top_lidar" parent="${prefix}front_case_link" prefix_topic="top_lidar" gpu="${gpu}">
       <origin xyz="${top_lidar_offset_x} ${top_lidar_offset_y} ${top_lidar_offset_z}" rpy="0 0 0"/>
-  </xacro:sensor_rslidar_16>
+  </xacro:sensor_rslidar_16> -->
   <xacro:sensor_sick_s300 prefix="${prefix}front_laser" parent="${prefix}front_case_link" prefix_topic="front_laser" min_angle="-2.35" max_angle="2.35" gpu="${gpu}" >
       <origin xyz="${front_laser_x} ${front_laser_y} ${front_laser_z}" rpy="${PI} 0 0"/>
   </xacro:sensor_sick_s300>
   <xacro:sensor_intel_d435 prefix="${prefix}left_fork_camera" parent="${prefix}left_fork_sensor_link" prefix_topic="${robot_id}/left_fork_camera" use_nominal_extrinsics="true" >
-        <origin xyz="0 0 0" rpy="0 -${5.0*PI/180.0} 0"/>
+        <origin xyz="0 0 0" rpy="0 0 0"/>
   </xacro:sensor_intel_d435>
   <xacro:sensor_intel_d435 prefix="${prefix}right_fork_camera" parent="${prefix}right_fork_sensor_link" prefix_topic="${robot_id}/right_fork_camera" use_nominal_extrinsics="true" >
